File: KicadJE_EffectsUnit2.kicad_pcb (KiCad board)
At the start: 2 copper layers, 100 x 100 mm, 70 parts, among them J201 In_1, J202 In 2, J203 Out 1, J204 Out 2, J205 Out Final, P201 Doepfer_Power_10pin, SW201 Out 1, SW202 In or cascade, SW203 Out 2 FB, SW204 In or cascade, SW205 HI/LO, U201 TL072, U202 TL072

Commit message: Routing of Distort2 done
Routing:
- net GND: track 38.5 -> 51.0 mm, vias 11 -> 83
- net (no net): vias 0 -> 1
- added copper zone on B.Cu, net GND
Changed lines of the file:
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@@
     (thickness 1.6)
     (drawings 27)
-    (tracks 510)
+    (tracks 586)
     (zones 0)
     (modules 70)
@@
   (gr_line (start 150 50) (end 150 150) (layer Edge.Cuts) (width 0.05))
   (gr_line (start 50 50) (end 150 50) (layer Edge.Cuts) (width 0.05))
+  (via (at 55 145) (size 0.7) (drill 0.4) (layers F.Cu B.Cu) (net 0))
+  (via (at 74 78) (size 0.7) (drill 0.4) (layers F.Cu B.Cu) (net 1))
+  (via (at 64 78) (size 0.7) (drill 0.4) (layers F.Cu B.Cu) (net 1))
+  (via (at 51 68) (size 0.7) (drill 0.4) (layers F.Cu B.Cu) (net 1))
+  (via (at 51 75) (size 0.7) (drill 0.4) (layers F.Cu B.Cu) (net 1))
   (segment (start 67.2 58.8) (end 67.96 58.04) (width 0.4) (layer F.Cu) (net 1))
   (segment (start 66 58.8) (end 67.2 58.8) (width 0.4) (layer F.Cu) (net 1))
@@
   (segment (start 76 126.525) (end 76 126.75) (width 0.4) (layer B.Cu) (net 1))
   (segment (start 76 126.75) (end 76.75 127.5) (width 0.4) (layer B.Cu) (net 1))
+  (via (at 87 139) (size 0.7) (drill 0.4) (layers F.Cu B.Cu) (net 1))
+  (via (at 69 131) (size 0.7) (drill 0.4) (layers F.Cu B.Cu) (net 1))
+  (via (at 76 131) (size 0.7) (drill 0.4) (layers F.Cu B.Cu) (net 1))
+  (via (at 64 131) (size 0.7) (drill 0.4) (layers F.Cu B.Cu) (net 1))
+  (via (at 55 131) (size 0.7) (drill 0.4) (layers F.Cu B.Cu) (net 1))
+  (via (at 55 125) (size 0.7) (drill 0.4) (layers F.Cu B.Cu) (net 1))
+  (via (at 55 119) (size 0.7) (drill 0.4) (layers F.Cu B.Cu) (net 1))
+  (via (at 67 119) (size 0.7) (drill 0.4) (layers F.Cu B.Cu) (net 1))
+  (via (at 71 119) (size 0.7) (drill 0.4) (layers F.Cu B.Cu) (net 1))
+  (via (at 71 115) (size 0.7) (drill 0.4) (layers F.Cu B.Cu) (net 1))
+  (via (at 67 113) (size 0.7) (drill 0.4) (layers F.Cu B.Cu) (net 1))
+  (via (at 57 109) (size 0.7) (drill 0.4) (layers F.Cu B.Cu) (net 1))
+  (via (at 55 109) (size 0.7) (drill 0.4) (layers F.Cu B.Cu) (net 1))
+  (via (at 57 112) (size 0.7) (drill 0.4) (layers F.Cu B.Cu) (net 1))
+  (via (at 67 103) (size 0.7) (drill 0.4) (layers F.Cu B.Cu) (net 1))
+  (via (at 71 103) (size 0.7) (drill 0.4) (layers F.Cu B.Cu) (net 1))
+  (via (at 71 94) (size 0.7) (drill 0.4) (layers F.Cu B.Cu) (net 1))
+  (via (at 63 90) (size 0.7) (drill 0.4) (layers F.Cu B.Cu) (net 1))
+  (via (at 69 78) (size 0.7) (drill 0.4) (layers F.Cu B.Cu) (net 1))
+  (via (at 69 68) (size 0.7) (drill 0.4) (layers F.Cu B.Cu) (net 1))
+  (via (at 69 52) (size 0.7) (drill 0.4) (layers F.Cu B.Cu) (net 1))
+  (via (at 59 60) (size 0.7) (drill 0.4) (layers F.Cu B.Cu) (net 1))
+  (via (at 79 60) (size 0.7) (drill 0.4) (layers F.Cu B.Cu) (net 1))
+  (via (at 87 67) (size 0.7) (drill 0.4) (layers F.Cu B.Cu) (net 1))
+  (via (at 87 75) (size 0.7) (drill 0.4) (layers F.Cu B.Cu) (net 1))
+  (segment (start 52 76) (end 51 75) (width 0.4) (layer F.Cu) (net 1))
+  (segment (start 52 80) (end 52 76) (width 0.4) (layer F.Cu) (net 1))
+  (segment (start 51 75) (end 51 68) (width 0.4) (layer F.Cu) (net 1))
+  (via (at 56 75) (size 0.7) (drill 0.4) (layers F.Cu B.Cu) (net 1))
+  (via (at 59 75) (size 0.7) (drill 0.4) (layers F.Cu B.Cu) (net 1))
+  (via (at 56 81) (size 0.7) (drill 0.4) (layers F.Cu B.Cu) (net 1))
+  (via (at 56 68) (size 0.7) (drill 0.4) (layers F.Cu B.Cu) (net 1))
+  (via (at 59 68) (size 0.7) (drill 0.4) (layers F.Cu B.Cu) (net 1))
+  (via (at 74 60) (size 0.7) (drill 0.4) (layers F.Cu B.Cu) (net 1))
+  (via (at 65 60) (size 0.7) (drill 0.4) (layers F.Cu B.Cu) (net 1))
+  (via (at 83 60) (size 0.7) (drill 0.4) (layers F.Cu B.Cu) (net 1))
+  (via (at 55 60) (size 0.7) (drill 0.4) (layers F.Cu B.Cu) (net 1))
+  (via (at 79 75) (size 0.7) (drill 0.4) (layers F.Cu B.Cu) (net 1))
+  (via (at 71 75) (size 0.7) (drill 0.4) (layers F.Cu B.Cu) (net 1))
+  (via (at 67 75) (size 0.7) (drill 0.4) (layers F.Cu B.Cu) (net 1))
+  (via (at 79 105) (size 0.7) (drill 0.4) (layers F.Cu B.Cu) (net 1))
+  (via (at 52 105) (size 0.7) (drill 0.4) (layers F.Cu B.Cu) (net 1))
+  (via (at 54 105) (size 0.7) (drill 0.4) (layers F.Cu B.Cu) (net 1))
+  (via (at 84 105) (size 0.7) (drill 0.4) (layers F.Cu B.Cu) (net 1))
+  (via (at 87 105) (size 0.7) (drill 0.4) (layers F.Cu B.Cu) (net 1))
+  (via (at 57 115) (size 0.7) (drill 0.4) (layers F.Cu B.Cu) (net 1))
+  (via (at 62 115) (size 0.7) (drill 0.4) (layers F.Cu B.Cu) (net 1))
+  (via (at 76 115) (size 0.7) (drill 0.4) (layers F.Cu B.Cu) (net 1))
+  (via (at 68 115) (size 0.7) (drill 0.4) (layers F.Cu B.Cu) (net 1))
+  (via (at 86 115) (size 0.7) (drill 0.4) (layers F.Cu B.Cu) (net 1))
+  (via (at 86 125) (size 0.7) (drill 0.4) (layers F.Cu B.Cu) (net 1))
+  (via (at 84 125) (size 0.7) (drill 0.4) (layers F.Cu B.Cu) (net 1))
+  (via (at 81 125) (size 0.7) (drill 0.4) (layers F.Cu B.Cu) (net 1))
+  (via (at 73 125) (size 0.7) (drill 0.4) (layers F.Cu B.Cu) (net 1))
+  (via (at 66 125) (size 0.7) (drill 0.4) (layers F.Cu B.Cu) (net 1))
+  (via (at 61 125) (size 0.7) (drill 0.4) (layers F.Cu B.Cu) (net 1))
+  (via (at 52 125) (size 0.7) (drill 0.4) (layers F.Cu B.Cu) (net 1))
+  (via (at 52 135) (size 0.7) (drill 0.4) (layers F.Cu B.Cu) (net 1))
+  (via (at 55 135) (size 0.7) (drill 0.4) (layers F.Cu B.Cu) (net 1))
+  (via (at 66 135) (size 0.7) (drill 0.4) (layers F.Cu B.Cu) (net 1))
+  (via (at 73 135) (size 0.7) (drill 0.4) (layers F.Cu B.Cu) (net 1))
+  (via (at 81 135) (size 0.7) (drill 0.4) (layers F.Cu B.Cu) (net 1))
+  (via (at 84 135) (size 0.7) (drill 0.4) (layers F.Cu B.Cu) (net 1))
+  (via (at 87 135) (size 0.7) (drill 0.4) (layers F.Cu B.Cu) (net 1))
+  (via (at 81 145) (size 0.7) (drill 0.4) (layers F.Cu B.Cu) (net 1))
+  (via (at 73 145) (size 0.7) (drill 0.4) (layers F.Cu B.Cu) (net 1))
+  (via (at 66 145) (size 0.7) (drill 0.4) (layers F.Cu B.Cu) (net 1))
+  (via (at 63 145) (size 0.7) (drill 0.4) (layers F.Cu B.Cu) (net 1))
+  (via (at 63 135) (size 0.7) (drill 0.4) (layers F.Cu B.Cu) (net 1))
+  (via (at 75 135) (size 0.7) (drill 0.4) (layers F.Cu B.Cu) (net 1))
+  (via (at 75 145) (size 0.7) (drill 0.4) (layers F.Cu B.Cu) (net 1))
   (segment (start 57.960001 89.485001) (end 57.975 89.5) (width 0.15) (layer B.Cu) (net 2))
   (segment (start 56.55 89.485001) (end 57.960001 89.485001) (width 0.15) (layer B.Cu) (net 2))
@@
     (connect_pads (clearance 0.508))
     (min_thickness 0.254)
+    (fill yes (arc_segments 32) (thermal_gap 0.508) (thermal_bridge_width 0.508))
+    (polygon
+      (pts
+        (xy 51 51) (xy 51 149) (xy 88 149) (xy 88 51)
+      )
+    )
+  )
+  (zone (net 1) (net_name GND) (layer B.Cu) (hatch edge 0.508)
+    (connect_pads (clearance 0.508))
+    (min_thickness 0.254)
