File: KicadJE_EffectsUnit2.kicad_pcb (KiCad board)
At the start: 2 copper layers, 100 x 100 mm, 161 parts, among them J201 In_1, J202 In 2, J203 Out 1, J204 Out 2, J205 Out Final, J301 Conn_01x09_Male, J302 Conn_01x09_Male, J401 Conn_01x09_Male, J402 Conn_01x09_Male, J403 Out 1, J404 In_1, J405 Out 2, J406 In 2, J407 Out 1 Final, J408 Out 2 Final, P201 Doepfer_Power_10pin, P301 Doepfer_Power_10pin, SW201 Out 1, SW202 In or cascade, SW203 Out 2 FB, SW204 In or cascade, SW205 HI/LO, U201 TL072, U202 TL072, U401 TL072, U402 TL072

Commit message: Update KicadJE_EffectsUnit2.kicad_pcb
Parts:
- moved R421 137.1 mm to (129.5, 164.0)
- moved D408 128.7 mm to (128.0, 157.0)
- moved C414 114.7 mm to (134.0, 164.0), turned to 180 degrees
- moved C408 112.4 mm to (125.5, 164.0), turned to 180 degrees
- moved R417 108.4 mm to (133.0, 158.0), turned to 90 degrees
- moved R413 103.6 mm to (120.0, 136.0), turned to 180 degrees
- moved D409 103.0 mm to (128.0, 161.0)
- moved R428 100.6 mm to (120.5, 119.5)
- moved R408 94.3 mm to (114.5, 82.5)
- moved R402 93.6 mm to (114.5, 73.5), turned to 180 degrees
- moved R416 92.8 mm to (121.0, 115.0)
- moved R403 83.4 mm to (120.2, 87.8)
- moved C401 81.1 mm to (117.8, 68.0), turned to 180 degrees
- moved R405 76.2 mm to (122.0, 68.0), turned to 180 degrees
- moved R409 75.9 mm to (118.2, 93.2)
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Connections:
- U401 pad 1: Net-(R405-Pad2) -> Net-(R404-Pad2)
- U401 pad 2: /KicadJE_EU8_Dist/POT1_L -> /KicadJE_EU8_Dist/POT2_L
- U401 pad 3: Net-(R407-Pad1) -> Net-(R408-Pad1)
- U401 pad 5: Net-(R408-Pad1) -> Net-(R407-Pad1)
- U401 pad 6: /KicadJE_EU8_Dist/POT2_L -> /KicadJE_EU8_Dist/POT1_L
- U401 pad 7: Net-(R404-Pad2) -> Net-(R405-Pad2)
- U402 pad 1: /KicadJE_EU8_Dist/POT3_C -> /KicadJE_EU8_Dist/POT4_C
- U402 pad 2: Net-(C407-Pad1) -> Net-(R413-Pad2)
- U402 pad 3: Net-(R418-Pad1) -> Net-(R419-Pad1)
- U402 pad 5: Net-(R419-Pad1) -> Net-(R418-Pad1)
- U402 pad 6: Net-(R413-Pad2) -> Net-(C407-Pad1)
- U402 pad 7: /KicadJE_EU8_Dist/POT4_C -> /KicadJE_EU8_Dist/POT3_C
Routing:
- net Net-(J404-PadTN): track 0.00 -> 53.4 mm
- net Net-(C409-Pad1): track 0.00 -> 34.4 mm
- net /KicadJE_EU8_Dist/POT1_L: track 0.00 -> 30.5 mm
- net /KicadJE_EU8_Dist/POT1_C: track 0.00 -> 19.5 mm
- net /KicadJE_EU8_Dist/POT2_L: track 0.00 -> 12.7 mm
- net Net-(R405-Pad2): track 0.00 -> 9.15 mm
- net Net-(C401-Pad2): track 0.00 -> 8.63 mm
- net Net-(J404-PadT): track 64.2 -> 70.6 mm
- net Out1_Dist: track 0.00 -> 3.90 mm
- net /KicadJE_EU8_Dist/POT2_C: track 0.00 -> 2.54 mm
- net Net-(C410-Pad1): track 12.2 -> 14.3 mm
- net Net-(R407-Pad1): track 31.5 -> 30.7 mm

Commit message: layers done
Parts:
- moved H403 143.1 mm to (142.2, 147.0)
- moved R423 108.1 mm to (115.0, 128.2), turned to 90 degrees
- moved H402 106.7 mm to (125.0, 147.0)
- moved R422 106.4 mm to (113.0, 128.2), turned to 90 degrees
- moved R419 102.9 mm to (115.0, 124.2), turned to 90 degrees
- moved R418 102.2 mm to (113.0, 124.2), turned to 90 degrees
- moved D411 90.1 mm to (139.5, 110.8)
- moved R420 89.8 mm to (122.2, 111.5)
- moved R412 87.9 mm to (118.0, 108.5), turned to 180 degrees
- moved R426 86.7 mm to (136.2, 107.5)
- moved R427 85.4 mm to (140.0, 107.5)
- moved D404 79.8 mm to (114.5, 93.2)
- moved R414 74.6 mm to (122.5, 102.0)
- moved R415 74.6 mm to (126.2, 102.0)
- moved D405 74.5 mm to (114.5, 96.8)
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Routing:
- net GND: track 79.6 -> 245.3 mm, vias 84 -> 118
- net Net-(R404-Pad2): track 0.00 -> 63.4 mm, vias 0 -> 1
- net /KicadJE_EU8_Dist/POT4_C: track 0.00 -> 48.4 mm, vias 0 -> 1
- net Net-(R413-Pad2): track 0.00 -> 32.1 mm, vias 0 -> 6
- net Net-(C411-Pad1): track 0.00 -> 31.0 mm
- net Net-(C407-Pad1): track 0.00 -> 28.1 mm
- net /KicadJE_EU8_Dist/POT3_C: track 0.00 -> 24.0 mm
- net /KicadJE_EU8_Dist/POT3_L: track 0.00 -> 22.4 mm
- net Out1_Final: track 0.00 -> 18.0 mm
- net Net-(R405-Pad2): track 9.15 -> 22.8 mm
- net Out2_Final: track 0.00 -> 13.4 mm
- net /KicadJE_EU8_Dist/POT2_C: track 2.54 -> 15.4 mm
- net Net-(C404-Pad1): track 0.00 -> 12.7 mm
- net Net-(C412-Pad1): track 0.00 -> 11.5 mm
- net Net-(R418-Pad1): track 0.00 -> 11.2 mm
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
Commit message: Labels and Text
Parts:
- added G***: LOGO, AJ:Johansen_engineering_logo_25mm_front_neg5, B.Cu at (139.0, 79.0)
- added G***: LOGO, AJ:Johansen_engineering_logo_25mm_front_neg5, B.Cu at (69.0, 140.0)
- added G***: LOGO, AJ:Johansen_engineering_logo_25mm_front_neg5, F.Cu at (95.0, 76.0)
- added G***: LOGO, AJ:Johansen_engineering_logo_25mm_front_neg5, F.Cu at (84.0, 76.0)
- added G***: LOGO, AJ:Johansen_engineering_logo_25mm_front_neg5, F.Cu at (130.0, 101.0)
Routing:
- net GND: track 245.3 -> 268.7 mm, vias 118 -> 121
- net Out2_Final: track 13.4 -> 15.1 mm
Other:
- board text added: "EU2-Dist1 Rev A - 15/09-2019"
- board text added: "EU2-Dist2 Rev A - 15/09-2019"
